File: electronics/KiCad/cascade_trigger.sch (KiCad schematic (older format))
At the start: 69 parts, among them J1 Power_In, J2 Conn_02x07_Odd_Even, U2 Teensy3.6

Commit message: clean up of old schematics and code
Parts:
- Driver_1, Driver_2, Driver_3, Driver_4, Driver_5, Driver_6, Driver_7, Driver_8: symbol custom_kicad_parts:EL7104 -> cascade_trigger-rescue:EL7104-custom_kicad_parts
- U2: symbol teensy:Teensy3.6 -> cascade_trigger-rescue:Teensy3.6-teensy
Other:
- moved on the sheet: R10, R11, R12, R13, Trig_IN_1, Trig_IN_2, Trig_IN_3, Trig_IN_4
